File: pcb/lmp91000-pcb.kicad_pcb (KiCad board)
At the start: 4 copper layers, 30 x 30 mm, 53 parts, among them J1 TC2030, J2 UJC-H-G-SMT-2-P6-TR, J3 0530480210, J4 TB0011-350-03GR, J5 0528070310, Q1 NTR4003N, SW1 PTS815SJM250SMTRLFS, U1 2450AT18D0100001E, U2 EFR32BG24L210F768IM40-B, U3 MCP73811T-420I-OT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

Commit message: Update back silkscreen with labels
Other:
- board text added: "v1.0"
